File: BFUSB_HUB.kicad_pcb (KiCad board)
At the start: 2 copper layers, 154.7 x 96 mm, 70 parts, among them J1 USB_C_Receptacle_USB2.0, J10 USB_A, J11 USB_A, J12 USB_A, J13 USB_A, J14 USB_A, J15 USB_A, J16 USB_A, J17 USB_A, J18 USB_A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

Commit message: added silksreen model number to board
Other:
- board text added: "BFUSB-16"
